Commit message: Finished model with visual and physical properties
Still missing Sensors and Gazebo link with joint controllers and transmission

File: jetsoncar_description/urdf/jetsoncar.xacro (robot description, xacro)
@@ -11,187 +11,248 @@
      and https://github.com/mit-racecar/racecar-simulator/blob/master/racecar_description/urdf/racecar.xacro
 -->
-	<xacro:property name="front_to_rear_wheel_center" value="0.42" />
-	<xacro:property name="left_to_right_wheel_center" value="0.285" />
-	<xacro:property name="baseplate_to_wheel_center" value="0.118" />
-	<xacro:property name="wheel_diameter" value="0.155" />
-	<xacro:property name="wheel_thickness" value="0.064" />
+	<!-- X axis direction is forward, Y axis direction is left -->
+	<xacro:include filename="$(find jetsoncar_description)/urdf/functions.xacro" />
 	<xacro:include filename="$(find jetsoncar_description)/urdf/materials.xacro" />
+	<xacro:include filename="$(find jetsoncar_description)/urdf/physical.xacro" />
+	<xacro:include filename="$(find jetsoncar_description)/urdf/joints.xacro" />
 	<link name="base_link" />
 	<link name="imu">
 		<visual>
-			<geometry>
-				<box size="0.05 0.05 0.03"/> <!-- 50x50x30 mm, Please confirm against 3D drawings -->
-			</geometry>
-			<origin xyz="0 0 0" rpy="0 0 0" /> <!-- origin (0,0,0) is in the center of the box -->
 			<material name="grey"/>
-		</visual>
-	</link>
+			<xacro:imu_geometry/>
+		</visual>
+		<collision>
+			<xacro:imu_geometry/>
+		</collision>
+		<inertial>
+			<xacro:imu_inertial/>
+		</inertial>
+	</link>
+	<xacro:fixed_offset_joint parent="baseplate" child="imu" offset="0 0 ${imu_height/2}"/> <!-- because origin is in the center, we want the IMU to stand on the baseplate -->
 	<link name="baseplate">
 		<visual>
-			<geometry>
-				<box size="0.50 0.20 0.0675"/> <!-- 50x20x6.75 cm, X-axis is front of vehicle -->
-			</geometry>
-			<origin xyz="0 0 0.03375" rpy="0 0 0" /> <!-- origin (0,0,0) is in the center of the box -->
 			<material name="acrylic"/>
-		</visual>
-	</link>
+			<xacro:baseplate_geometry/>
+		</visual>
+		<collision>
+			<xacro:baseplate_geometry/>
+		</collision>
+		<inertial>
+			<xacro:baseplate_inertial/>
+		</inertial>
+	</link>
+	<xacro:fixed_offset_joint parent="base_link" child="baseplate" offset="0 0 0"/>
 	<link name="front_mount">
 		<visual>
-			<geometry>
-				<box size="0.24 0.12 0.01"/>
-			</geometry>
-			<origin xyz="0 0 0" rpy="0 0.5 0" /> <!-- origin (0,0,0) is in the center of the box -->
 			<material name="grey"/>
-		</visual>
-	</link>
+			<xacro:front_mount_geometry/>
+		</visual>
+		<collision>
+			<xacro:front_mount_geometry/>
+		</collision>
+		<inertial>
+			<xacro:front_mount_inertial/>
+		</inertial>
+	</link>
+	<xacro:fixed_offset_joint parent="baseplate" child="front_mount" offset="${front_to_rear_wheel_center/4} 0 -${baseplate_to_wheel_center/2}"/>
 	<link name="rear_mount">
 		<visual>
-			<geometry>
-				<box size="0.24 0.12 0.01"/>
-			</geometry>
-			<origin xyz="0 0 0" rpy="0 -0.5 0" /> <!-- origin (0,0,0) is in the center of the box -->
 			<material name="grey"/>
-		</visual>
-	</link>
+			<xacro:rear_mount_geometry/>
+		</visual>
+		<collision>
+			<xacro:rear_mount_geometry/>
+		</collision>
+		<inertial>
+			<xacro:rear_mount_inertial/>
+		</inertial>
+	</link>
+	<xacro:fixed_offset_joint parent="baseplate" child="rear_mount" offset="-${front_to_rear_wheel_center/4} 0 -${baseplate_to_wheel_center/2}"/>
+	<link name="front_shaft">
+		<visual>
+			<material name="black"/>
+			<xacro:shaft_geometry/>
+		</visual>
+		<collision>
+			<xacro:shaft_geometry/>
+		</collision>
+		<inertial>
+			<xacro:shaft_inertial/>
+		</inertial>
+	</link>
+	<xacro:fixed_offset_joint parent="front_mount" child="front_shaft" offset="${front_to_rear_wheel_center/4} 0 -${baseplate_to_wheel_center/2}"/>
 	<link name="rear_shaft">
 		<visual>
-			<geometry>
-				<cylinder length="${left_to_right_wheel_center}" radius="0.018"/> <!-- confirm length between wheels -->
-			</geometry>
-			<origin xyz="0 0 0" rpy="1.570796327 0 0" /> <!-- origin (0,0,0) is in the center of the cylinder -->
-			<material name="black"/>
-		</visual>
-	</link>
-	<link name="front_shaft">
-		<visual>
-			<geometry>
-				<cylinder length="${left_to_right_wheel_center}" radius="0.018"/> <!-- confirm length between wheels -->
-			</geometry>
-			<origin xyz="0 0 0" rpy="1.570796327 0 0" /> <!-- origin (0,0,0) is in the center of the cylinder -->
-			<material name="black"/>
-		</visual>
-	</link>
+			<material name="black"/>
+			<xacro:shaft_geometry/>
+		</visual>
+		<collision>
+			<xacro:shaft_geometry/>
+		</collision>
+		<inertial>
+			<xacro:shaft_inertial/>
+		</inertial>
+	</link>
+	<xacro:fixed_offset_joint parent="rear_mount" child="rear_shaft" offset="-${front_to_rear_wheel_center/4} 0 -${baseplate_to_wheel_center/2}"/>
 	<link name="front_right_bearing">
 		<visual>
-			<geometry>
-				<sphere radius="0.015"/>
-			</geometry>
-			<origin xyz="0 0 0" rpy="0 0 0" /> <!-- origin (0,0,0) is in the center of the cylinder -->
 			<material name="white"/>
-		</visual>
+			<xacro:bearing_geometry/>
+		</visual>
+		<collision>
+			<xacro:bearing_geometry/>
+		</collision>
+		<inertial>
+			<xacro:bearing_inertial/>
+		</inertial>
+	</link>
+	<link name="front_left_bearing">
+		<visual>
+			<material name="white"/>
+			<xacro:bearing_geometry/>
+		</visual>
+		<collision>
+			<xacro:bearing_geometry/>
+		</collision>
+		<inertial>
+			<xacro:bearing_inertial/>
+		</inertial>
 	</link>
 	<link name="front_right_wheel">
 		<visual>
-			<geometry>
-				<cylinder length="${wheel_thickness}" radius="${wheel_diameter/2}"/>
-			</geometry>
-			<origin xyz="0 0 0" rpy="1.570796327 0 0" /> <!-- origin (0,0,0) is in the center of the cylinder -->
-			<material name="black"/>
-		</visual>
-	</link>
-	<link name="front_left_bearing">
-		<visual>
-			<geometry>
-				<sphere radius="0.015"/>
-			</geometry>
-			<origin xyz="0 0 0" rpy="0 0 0" /> <!-- origin (0,0,0) is in the center of the cylinder -->
-			<material name="white"/>
-		</visual>
+			<material name="black"/>
+			<xacro:wheel_geometry/>
+		</visual>
+		<collision>
+			<xacro:wheel_geometry/>
+			<contact_coefficients mu="0" kp="1000.0" kd="1.0"/>  <!-- mu=The friction coefficient, kp=Stiffness coefficient, kd=Dampening coefficient -->
+		</collision>
+		<inertial>
+			<xacro:wheel_inertial/>
+		</inertial>
 	</link>
 	<link name="front_left_wheel">
 		<visual>
-			<geometry>
-				<cylinder length="${wheel_thickness}" radius="${wheel_diameter/2}"/>
-			</geometry>
-			<origin xyz="0 0 0" rpy="1.570796327 0 0" /> <!-- origin (0,0,0) is in the center of the cylinder -->
-			<material name="black"/>
-		</visual>
+			<material name="black"/>
+			<xacro:wheel_geometry/>
+		</visual>
+		<collision>
+			<xacro:wheel_geometry/>
+			<contact_coefficients mu="0" kp="1000.0" kd="1.0"/>  <!-- mu=The friction coefficient, kp=Stiffness coefficient, kd=Dampening coefficient -->
+		</collision>
+		<inertial>
+			<xacro:wheel_inertial/>
+		</inertial>
 	</link>
 	<link name="rear_right_wheel">
 		<visual>
-			<geometry>
-				<cylinder length="${wheel_thickness}" radius="${wheel_diameter/2}"/>
-			</geometry>
-			<origin xyz="0 0 0" rpy="1.570796327 0 0" /> <!-- origin (0,0,0) is in the center of the cylinder -->
-			<material name="black"/>
-		</visual>
+			<material name="black"/>
+			<xacro:wheel_geometry/>
+		</visual>
+		<collision>
+			<xacro:wheel_geometry/>
+			<contact_coefficients mu="0" kp="1000.0" kd="1.0"/>  <!-- mu=The friction coefficient, kp=Stiffness coefficient, kd=Dampening coefficient -->
+		</collision>
+		<inertial>
+			<xacro:wheel_inertial/>
+		</inertial>
 	</link>
 	<link name="rear_left_wheel">
 		<visual>
-			<geometry>
-				<cylinder length="${wheel_thickness}" radius="${wheel_diameter/2}"/>
-			</geometry>
-			<origin xyz="0 0 0" rpy="1.570796327 0 0" /> <!-- origin (0,0,0) is in the center of the cylinder -->
-			<material name="black"/>
-		</visual>
-	</link>
-	<joint name="baselink_to_baseplate" type="fixed">
-		<parent link="base_link"/>
-		<child link="baseplate"/>
-		<origin xyz="0 0 0" rpy="0 0 0" /> <!-- offset from parent to child, so with direction based in parent frame -->
-	</joint>
-	<joint name="baseplate_to_imu" type="fixed">
-		<parent link="baseplate"/>
-		<child link="imu"/>
-		<origin xyz="0 0 0.015" rpy="0 0 0" /> <!-- offset from parent to child, so with direction based in parent frame -->
-	</joint>
-	<joint name="baseplate_to_front_mount" type="fixed">
-		<parent link="baseplate"/>
-		<child link="front_mount"/>
-		<origin xyz="${front_to_rear_wheel_center/4} 0 -${baseplate_to_wheel_center/2}" rpy="0 0 0" /> <!-- offset from parent to child, so with direction based in parent frame -->
-	</joint>
-	<joint name="front_mount_to_front_shaft" type="fixed">
-		<parent link="front_mount"/>
-		<child link="front_shaft"/>
-		<origin xyz="${front_to_rear_wheel_center/4} 0 -${baseplate_to_wheel_center/2}" rpy="0 0 0" /> <!-- offset from parent to child, so with direction based in parent frame -->
-	</joint>
-	<joint name="baseplate_to_rear_mount" type="fixed">
-		<parent link="baseplate"/>
-		<child link="rear_mount"/>
-		<origin xyz="-${front_to_rear_wheel_center/4} 0 -${baseplate_to_wheel_center/2}" rpy="0 0 0" /> <!-- offset from parent to child, so with direction based in parent frame -->
-	</joint>
-	<joint name="rear_mount_to_rear_shaft" type="fixed">
-		<parent link="rear_mount"/>
-		<child link="rear_shaft"/>
-		<origin xyz="-${front_to_rear_wheel_center/4} 0 -${baseplate_to_wheel_center/2}" rpy="0 0 0" /> <!-- offset from parent to child, so with direction based in parent frame -->
-	</joint>
-	<joint name="front_right_bearing_joint" type="revolute"> <!-- revolute is a joint with a range limited motion around its' axis -->
-		<parent link="front_shaft"/>
-		<child link="front_right_bearing"/>
-		<origin xyz="0 -${left_to_right_wheel_center/2} 0" rpy="0 0 0" /> <!-- offset from parent to child, so with direction based in parent frame -->
-		<axis xyz="0 0 1"/>
-    		<limit lower="-${20/180*pi}" upper="${20/180*pi}" effort="1000" velocity="0.5"/>
-	</joint>
-	<joint name="front_right_wheel_joint" type="continuous"> <!-- continuous is a joint of continous motion around its' axis -->
-		<parent link="front_right_bearing"/>
-		<child link="front_right_wheel"/>
-		<origin xyz="0 0 0" rpy="0 0 0" /> <!-- offset from parent to child, so with direction based in parent frame -->
-		<axis xyz="0 1 0"/>
-	</joint>
-	<joint name="front_left_bearing_joint" type="revolute"> <!-- revolute is a joint with a range limited motion around its' axis -->
-		<parent link="front_shaft"/>
-		<child link="front_left_bearing"/>
-		<origin xyz="0 ${left_to_right_wheel_center/2} 0" rpy="0 0 0" /> <!-- offset from parent to child, so with direction based in parent frame -->
-		<axis xyz="0 0 1"/>
-    		<limit lower="-${20/180*pi}" upper="${20/180*pi}" effort="1000" velocity="0.5"/>
-	</joint>
-	<joint name="front_left_wheel_joint" type="continuous"> <!-- continuous is a joint of continous motion around its' axis -->
-		<parent link="front_left_bearing"/>
-		<child link="front_left_wheel"/>
-		<origin xyz="0 0 0" rpy="0 0 0" /> <!-- offset from parent to child, so with direction based in parent frame -->
-		<axis xyz="0 1 0"/>
-	</joint>
-	<joint name="rear_right_wheel_joint" type="continuous"> <!-- continuous is a joint of continous motion around its' axis -->
-		<parent link="rear_shaft"/>
-		<child link="rear_right_wheel"/>
-		<origin xyz="0 -${left_to_right_wheel_center/2} 0" rpy="0 0 0" /> <!-- offset from parent to child, so with direction based in parent frame -->
-		<axis xyz="0 1 0"/>
-	</joint>
-	<joint name="rear_left_wheel_joint" type="continuous"> <!-- continuous is a joint of continous motion around its' axis -->
-		<parent link="rear_shaft"/>
-		<child link="rear_left_wheel"/>
-		<origin xyz="0 ${left_to_right_wheel_center/2} 0" rpy="0 0 0" /> <!-- offset from parent to child, so with direction based in parent frame -->
-		<axis xyz="0 1 0"/>
-	</joint>
+			<material name="black"/>
+			<xacro:wheel_geometry/>
+		</visual>
+		<collision>
+			<xacro:wheel_geometry/>
+			<contact_coefficients mu="0" kp="1000.0" kd="1.0"/>  <!-- mu=The friction coefficient, kp=Stiffness coefficient, kd=Dampening coefficient -->
+		</collision>
+		<inertial>
+			<xacro:wheel_inertial/>
+		</inertial>
+	</link>
+	<xacro:steering_joint parent="front_shaft" child="front_right_bearing" offset="0 -${left_to_right_wheel_center/2} 0"/>
+	<xacro:steering_joint parent="front_shaft" child="front_left_bearing" offset="0 ${left_to_right_wheel_center/2} 0"/>
+	<xacro:wheel_joint parent="front_right_bearing" child="front_right_wheel" offset="0 0 0"/>
+	<xacro:wheel_joint parent="front_left_bearing" child="front_left_wheel" offset="0 0 0"/>
+	<xacro:wheel_joint parent="rear_shaft" child="rear_right_wheel" offset="0 -${left_to_right_wheel_center/2} 0"/>
+	<xacro:wheel_joint parent="rear_shaft" child="rear_left_wheel" offset="0 ${left_to_right_wheel_center/2} 0"/>
+	<link name="left_camera_mount">
+		<visual>
+			<material name="blue"/>
+			<xacro:camera_mount_geometry/>
+		</visual>
+		<collision>
+			<xacro:camera_mount_geometry/>
+		</collision>
+		<inertial>
+			<xacro:camera_mount_inertial/>
+		</inertial>
+	</link>
+	<xacro:fixed_offset_joint parent="baseplate" child="left_camera_mount" offset="${baseplate_length/2-baseplate_frontedge_to_camera} ${camera_disparity/2} ${baseplate_thickness}"/>
+	<link name="left_camera">
+		<visual>
+			<material name="blue"/>
+			<xacro:camera_geometry/>
+		</visual>
+		<collision>
+			<xacro:camera_geometry/>
+		</collision>
+		<inertial>
+			<xacro:camera_inertial/>
+		</inertial>
+	</link>
+	<xacro:fixed_offset_joint parent="left_camera_mount" child="left_camera" offset="0 0 ${camera_mount_height+camera_height/2}"/>
+	<link name="right_camera_mount">
+		<visual>
+			<material name="blue"/>
+			<xacro:camera_mount_geometry/>
+		</visual>
+		<collision>
+			<xacro:camera_mount_geometry/>
+		</collision>
+		<inertial>
+			<xacro:camera_mount_inertial/>
+		</inertial>
+	</link>
+	<xacro:fixed_offset_joint parent="baseplate" child="right_camera_mount" offset="${baseplate_length/2-baseplate_frontedge_to_camera} -${camera_disparity/2} ${baseplate_thickness}"/>
+	<link name="right_camera">
+		<visual>
+			<material name="blue"/>
+			<xacro:camera_geometry/>
+		</visual>
+		<collision>
+			<xacro:camera_geometry/>
+		</collision>
+		<inertial>
+			<xacro:camera_inertial/>
+		</inertial>
+	</link>
+	<xacro:fixed_offset_joint parent="right_camera_mount" child="right_camera" offset="0 0 ${camera_mount_height+camera_height/2}"/>
+	<link name="lidar_mount">
+		<visual>
+			<material name="red"/>
+			<xacro:lidar_mount_geometry/>
+		</visual>
+		<collision>
+			<xacro:lidar_mount_geometry/>
+		</collision>
+		<inertial>
+			<xacro:lidar_mount_inertial/>
+		</inertial>
+	</link>
+	<xacro:fixed_offset_joint parent="baseplate" child="lidar_mount" offset="0 0 ${baseplate_thickness}"/>
+	<link name="lidar">
+		<visual>
+			<material name="red"/>
+			<xacro:lidar_geometry/>
+		</visual>
+		<collision>
+			<xacro:lidar_geometry/>
+		</collision>
+		<inertial>
+			<xacro:lidar_inertial/>
+		</inertial>
+	</link>
+	<xacro:fixed_offset_joint parent="lidar_mount" child="lidar" offset="0 0 ${lidar_mount_height}"/>
 	<xacro:include filename="$(find jetsoncar_description)/urdf/gazebo.xacro" />
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