Commit message: Included Gazebo launch files and configuration with joint controllers
OBS. The cars spawn inside the ground. I don't know why?

File: jetsoncar_description/urdf/functions.xacro (robot description, xacro)
@@ -3,5 +3,5 @@
 	<!-- Based on https://en.wikipedia.org/wiki/List_of_moments_of_inertia -->
 	<xacro:macro name="box_inertial" params="mass width length height">
-		<mass value="1e-5" />
+		<mass value="${mass}" />
 		<inertia ixx="${1/12*mass*(width*width+height*height)}"
 			 ixy="0"
@@ -13,5 +13,5 @@
 	</xacro:macro>
 	<xacro:macro name="cylinder_inertial" params="mass radius length">
-		<mass value="1e-5" />
+		<mass value="${mass}" />
 		<inertia ixx="${1/12*mass*(3*radius*radius+length*length)}"
 			 ixy="0"

File: jetsoncar_description/urdf/gazebo.xacro (robot description, xacro)
@@ -1,5 +1,163 @@
 <?xml version="1.0"?>
 <robot name="jetsoncar" xmlns:xacro="http://www.ros.org/wiki/xacro">
-<!-- include the Gazebo description of the JetsonCar -->
-<!-- eg. inspired from the racecar project or https://github.com/husky/husky_simulator/blob/indigo-devel/husky_gazebo/urdf/husky.gazebo.xacro -->
+	<!-- include the Gazebo description of the JetsonCar -->
+	<!-- see the guide: http://wiki.ros.org/urdf/Tutorials/Using%20a%20URDF%20in%20Gazebo -->
+	<!-- inspired from https://github.com/mit-racecar/racecar-simulator/blob/master/racecar_description/urdf/racecar.gazebo and https://github.com/husky/husky_simulator/blob/indigo-devel/husky_gazebo/urdf/husky.gazebo.xacro -->
+	<!-- We need to link Gazebo and ROS and let Gazebo load all the previously defined ROS parameters. Therefore this Gazebo file should be included in the end of the main xacro file! -->
+	<!-- Link Gazebo and ROS -->
+	<gazebo>
+		<plugin name="gazebo_ros_control" filename="libgazebo_ros_control.so">
+			<robotNamespace>/jetsoncar</robotNamespace>
+			<!--<robotSimType>gazebo_ros_control/DefaultRobotHWSim</robotSimType> -->
+		</plugin>
+	</gazebo>
+	<!-- Visual and physical properties -->
+	<!-- See http://gazebosim.org/tutorials?tut=ros_urdf&cat=connect_ros -->
+	<gazebo reference="baseplate">
+		<material>Gazebo/Grey</material>
+		<mu1 value="0.0"/> <!-- Columb friction coefficient in fdir1 direction -->
+		<mu2 value="0.0"/> <!-- Columb friction in perpendicular direction to fdir1 -->
+		<fdir1 value="1 0 0"/> <!-- direction of mu1 friction coefficient in the collision frame -->
+		<kp  value="10000000.0" /> <!-- contact stiffness -->
+		<kd  value="1.0" /> <!-- contact damping -->
+		<turnGravityOff>false</turnGravityOff>
+	</gazebo>
+	<gazebo reference="imu">
+		<material>Gazebo/Grey</material>
+		<mu1 value="0.0"/> <!-- Columb friction coefficient in fdir1 direction -->
+		<mu2 value="0.0"/> <!-- Columb friction in perpendicular direction to fdir1 -->
+		<fdir1 value="1 0 0"/> <!-- direction of mu1 friction coefficient in the collision frame -->
+		<kp  value="10000000.0" /> <!-- contact stiffness -->
+		<kd  value="1.0" /> <!-- contact damping -->
+		<turnGravityOff>false</turnGravityOff>
+	</gazebo>
+	<gazebo reference="front_mount">
+		<material>Gazebo/Grey</material>
+		<mu1 value="0.0"/> <!-- Columb friction coefficient in fdir1 direction -->
+		<mu2 value="0.0"/> <!-- Columb friction in perpendicular direction to fdir1 -->
+		<fdir1 value="1 0 0"/> <!-- direction of mu1 friction coefficient in the collision frame -->
+		<kp  value="10000000.0" /> <!-- contact stiffness -->
+		<kd  value="1.0" /> <!-- contact damping -->
+		<turnGravityOff>false</turnGravityOff>
+	</gazebo>
+	<gazebo reference="rear_mount">
+		<material>Gazebo/Grey</material>
+		<mu1 value="0.0"/> <!-- Columb friction coefficient in fdir1 direction -->
+		<mu2 value="0.0"/> <!-- Columb friction in perpendicular direction to fdir1 -->
+		<fdir1 value="1 0 0"/> <!-- direction of mu1 friction coefficient in the collision frame -->
+		<kp  value="10000000.0" /> <!-- contact stiffness -->
+		<kd  value="1.0" /> <!-- contact damping -->
+		<turnGravityOff>false</turnGravityOff>
+	</gazebo>
+	<gazebo reference="front_shaft">
+		<material>Gazebo/Black</material>
+		<mu1 value="0.0"/> <!-- Columb friction coefficient in fdir1 direction -->
+		<mu2 value="0.0"/> <!-- Columb friction in perpendicular direction to fdir1 -->
+		<fdir1 value="1 0 0"/> <!-- direction of mu1 friction coefficient in the collision frame -->
+		<kp  value="10000000.0" /> <!-- contact stiffness -->
+		<kd  value="1.0" /> <!-- contact damping -->
+		<turnGravityOff>false</turnGravityOff>
+	</gazebo>
+	<gazebo reference="rear_shaft">
+		<material>Gazebo/Black</material>
+		<mu1 value="0.0"/> <!-- Columb friction coefficient in fdir1 direction -->
+		<mu2 value="0.0"/> <!-- Columb friction in perpendicular direction to fdir1 -->
+		<fdir1 value="1 0 0"/> <!-- direction of mu1 friction coefficient in the collision frame -->
+		<kp  value="10000000.0" /> <!-- contact stiffness -->
+		<kd  value="1.0" /> <!-- contact damping -->
+		<turnGravityOff>false</turnGravityOff>
+	</gazebo>
+	<gazebo reference="front_right_wheel">
+		<material>Gazebo/Black</material>
+		<mu1 value="1.0"/> <!-- Columb friction coefficient in fdir1 direction -->
+		<mu2 value="1.0"/> <!-- Columb friction in perpendicular direction to fdir1 -->
+		<fdir1 value="1 0 0"/> <!-- direction of mu1 friction coefficient in the collision frame -->
+		<kp  value="10000000.0" /> <!-- contact stiffness -->
+		<kd  value="1.0" /> <!-- contact damping -->
+		<turnGravityOff>false</turnGravityOff>
+	</gazebo>
+	<gazebo reference="front_left_wheel">
+		<material>Gazebo/Black</material>
+		<mu1 value="1.0"/> <!-- Columb friction coefficient in fdir1 direction -->
+		<mu2 value="1.0"/> <!-- Columb friction in perpendicular direction to fdir1 -->
+		<fdir1 value="1 0 0"/> <!-- direction of mu1 friction coefficient in the collision frame -->
+		<kp  value="10000000.0" /> <!-- contact stiffness -->
+		<kd  value="1.0" /> <!-- contact damping -->
+		<turnGravityOff>false</turnGravityOff>
+	</gazebo>
+	<gazebo reference="rear_right_wheel">
+		<material>Gazebo/Black</material>
+		<mu1 value="1.0"/> <!-- Columb friction coefficient in fdir1 direction -->
+		<mu2 value="1.0"/> <!-- Columb friction in perpendicular direction to fdir1 -->
+		<fdir1 value="1 0 0"/> <!-- direction of mu1 friction coefficient in the collision frame -->
+		<kp  value="10000000.0" /> <!-- contact stiffness -->
+		<kd  value="1.0" /> <!-- contact damping -->
+		<turnGravityOff>false</turnGravityOff>
+	</gazebo>
+	<gazebo reference="rear_left_wheel">
+		<material>Gazebo/Black</material>
+		<mu1 value="1.0"/> <!-- Columb friction coefficient in fdir1 direction -->
+		<mu2 value="1.0"/> <!-- Columb friction in perpendicular direction to fdir1 -->
+		<fdir1 value="1 0 0"/> <!-- direction of mu1 friction coefficient in the collision frame -->
+		<kp  value="10000000.0" /> <!-- contact stiffness -->
+		<kd  value="1.0" /> <!-- contact damping -->
+		<turnGravityOff>false</turnGravityOff>
+	</gazebo>
+	<gazebo reference="lidar_mount">
+		<material>Gazebo/Red</material>
+		<mu1 value="0.0"/> <!-- Columb friction coefficient in fdir1 direction -->
+		<mu2 value="0.0"/> <!-- Columb friction in perpendicular direction to fdir1 -->
+		<fdir1 value="1 0 0"/> <!-- direction of mu1 friction coefficient in the collision frame -->
+		<kp  value="10000000.0" /> <!-- contact stiffness -->
+		<kd  value="1.0" /> <!-- contact damping -->
+		<turnGravityOff>false</turnGravityOff>
+	</gazebo>
+	<gazebo reference="lidar">
+		<material>Gazebo/Black</material>
+		<mu1 value="0.0"/> <!-- Columb friction coefficient in fdir1 direction -->
+		<mu2 value="0.0"/> <!-- Columb friction in perpendicular direction to fdir1 -->
+		<fdir1 value="1 0 0"/> <!-- direction of mu1 friction coefficient in the collision frame -->
+		<kp  value="10000000.0" /> <!-- contact stiffness -->
+		<kd  value="1.0" /> <!-- contact damping -->
+		<turnGravityOff>false</turnGravityOff>
+	</gazebo>
+	<gazebo reference="left_camera_mount">
+		<material>Gazebo/Black</material>
+		<mu1 value="0.0"/> <!-- Columb friction coefficient in fdir1 direction -->
+		<mu2 value="0.0"/> <!-- Columb friction in perpendicular direction to fdir1 -->
+		<fdir1 value="1 0 0"/> <!-- direction of mu1 friction coefficient in the collision frame -->
+		<kp  value="10000000.0" /> <!-- contact stiffness -->
+		<kd  value="1.0" /> <!-- contact damping -->
+		<turnGravityOff>false</turnGravityOff>
+	</gazebo>
+	<gazebo reference="left_camera">
+		<material>Gazebo/Blue</material>
+		<mu1 value="0.0"/> <!-- Columb friction coefficient in fdir1 direction -->
+		<mu2 value="0.0"/> <!-- Columb friction in perpendicular direction to fdir1 -->
+		<fdir1 value="1 0 0"/> <!-- direction of mu1 friction coefficient in the collision frame -->
+		<kp  value="10000000.0" /> <!-- contact stiffness -->
+		<kd  value="1.0" /> <!-- contact damping -->
+		<turnGravityOff>false</turnGravityOff>
+	</gazebo>
+	<gazebo reference="right_camera_mount">
+		<material>Gazebo/Black</material>
+		<mu1 value="0.0"/> <!-- Columb friction coefficient in fdir1 direction -->
+		<mu2 value="0.0"/> <!-- Columb friction in perpendicular direction to fdir1 -->
+		<fdir1 value="1 0 0"/> <!-- direction of mu1 friction coefficient in the collision frame -->
+		<kp  value="10000000.0" /> <!-- contact stiffness -->
+		<kd  value="1.0" /> <!-- contact damping -->
+		<turnGravityOff>false</turnGravityOff>
+	</gazebo>
+	<gazebo reference="right_camera">
+		<material>Gazebo/Blue</material>
+		<mu1 value="0.0"/> <!-- Columb friction coefficient in fdir1 direction -->
+		<mu2 value="0.0"/> <!-- Columb friction in perpendicular direction to fdir1 -->
+		<fdir1 value="1 0 0"/> <!-- direction of mu1 friction coefficient in the collision frame -->
+		<kp  value="10000000.0" /> <!-- contact stiffness -->
+		<kd  value="1.0" /> <!-- contact damping -->
+		<turnGravityOff>false</turnGravityOff>
+	</gazebo>
+	<!-- Plugins, eg. sensors -->
+	<!-- hokuyo LiDAR can be found here: https://github.com/mit-racecar/racecar-simulator/blob/master/racecar_description/urdf/racecar.gazebo#L59 -->
+	<!-- camera sensor might be found here: https://github.com/JoshMarino/gazebo_and_ros_control or here: http://gazebosim.org/tutorials?tut=ros_gzplugins -->
 </robot>

File: jetsoncar_description/urdf/jetsoncar.xacro (robot description, xacro)
@@ -16,4 +16,5 @@
 	<xacro:include filename="$(find jetsoncar_description)/urdf/physical.xacro" />
 	<xacro:include filename="$(find jetsoncar_description)/urdf/joints.xacro" />
+	<xacro:include filename="$(find jetsoncar_description)/urdf/transmissions.xacro" />
 	<link name="base_link" />
 	<link name="imu">
@@ -82,4 +83,5 @@
 	</link>
 	<xacro:fixed_offset_joint parent="front_mount" child="front_shaft" offset="${front_to_rear_wheel_center/4} 0 -${baseplate_to_wheel_center/2}"/>
+	<!--<xacro:dampener_joint parent="front_mount" child="front_shaft" offset="${front_to_rear_wheel_center/4} 0 -${baseplate_to_wheel_center/2}"/> I can not get the dampener joint to work properly. The car seems to be bouncing around, like the spring is too hard and dampening is too little. I already tried adjusting several parameters. -->
 	<link name="rear_shaft">
 		<visual>
@@ -95,28 +97,31 @@
 	</link>
 	<xacro:fixed_offset_joint parent="rear_mount" child="rear_shaft" offset="-${front_to_rear_wheel_center/4} 0 -${baseplate_to_wheel_center/2}"/>
-	<link name="front_right_bearing">
+	<!-- <xacro:dampener_joint parent="rear_mount" child="rear_shaft" offset="-${front_to_rear_wheel_center/4} 0 -${baseplate_to_wheel_center/2}"/> I can not get the dampener joint to work properly. The car seems to be bouncing around, like the spring is too hard and dampening is too little. I already tried adjusting several parameters. -->
+	<link name="front_right_hinge">
 		<visual>
 			<material name="white"/>
-			<xacro:bearing_geometry/>
-		</visual>
-		<collision>
-			<xacro:bearing_geometry/>
-		</collision>
-		<inertial>
-			<xacro:bearing_inertial/>
-		</inertial>
-	</link>
-	<link name="front_left_bearing">
+			<xacro:hinge_geometry/>
+		</visual>
+		<collision>
+			<xacro:hinge_geometry/>
+		</collision>
+		<inertial>
+			<xacro:hinge_inertial/>
+		</inertial>
+	</link>
+	<xacro:hinge_joint parent="front_shaft" child="front_right_hinge" offset="0 -${left_to_right_wheel_center/2} 0"/>
+	<link name="front_left_hinge">
 		<visual>
 			<material name="white"/>
-			<xacro:bearing_geometry/>
-		</visual>
-		<collision>
-			<xacro:bearing_geometry/>
-		</collision>
-		<inertial>
-			<xacro:bearing_inertial/>
-		</inertial>
-	</link>
+			<xacro:hinge_geometry/>
+		</visual>
+		<collision>
+			<xacro:hinge_geometry/>
+		</collision>
+		<inertial>
+			<xacro:hinge_inertial/>
+		</inertial>
+	</link>
+	<xacro:hinge_joint parent="front_shaft" child="front_left_hinge" offset="0 ${left_to_right_wheel_center/2} 0"/>
 	<link name="front_right_wheel">
 		<visual>
@@ -132,4 +137,5 @@
 		</inertial>
 	</link>
+	<xacro:wheel_joint parent="front_right_hinge" child="front_right_wheel" offset="0 0 0"/>
 	<link name="front_left_wheel">
 		<visual>
@@ -145,4 +151,5 @@
 		</inertial>
 	</link>
+	<xacro:wheel_joint parent="front_left_hinge" child="front_left_wheel" offset="0 0 0"/>
 	<link name="rear_right_wheel">
 		<visual>
@@ -158,4 +165,5 @@
 		</inertial>
 	</link>
+	<xacro:wheel_joint parent="rear_shaft" child="rear_right_wheel" offset="0 -${left_to_right_wheel_center/2} 0"/>
 	<link name="rear_left_wheel">
 		<visual>
@@ -171,10 +179,13 @@
 		</inertial>
 	</link>
-	<xacro:steering_joint parent="front_shaft" child="front_right_bearing" offset="0 -${left_to_right_wheel_center/2} 0"/>
-	<xacro:steering_joint parent="front_shaft" child="front_left_bearing" offset="0 ${left_to_right_wheel_center/2} 0"/>
-	<xacro:wheel_joint parent="front_right_bearing" child="front_right_wheel" offset="0 0 0"/>
-	<xacro:wheel_joint parent="front_left_bearing" child="front_left_wheel" offset="0 0 0"/>
-	<xacro:wheel_joint parent="rear_shaft" child="rear_right_wheel" offset="0 -${left_to_right_wheel_center/2} 0"/>
 	<xacro:wheel_joint parent="rear_shaft" child="rear_left_wheel" offset="0 ${left_to_right_wheel_center/2} 0"/>
+	<!-- Transmissions are motors attached to a certain joint. We thus need to instantiate transmissions at the corresponding joints -->
+	<xacro:wheel_transmission wheel="front_right_wheel"/>
+	<xacro:wheel_transmission wheel="front_left_wheel"/>
+	<!--<xacro:wheel_transmission wheel="rear_right_wheel"/>    Currently only front wheel drive!
+	<xacro:wheel_transmission wheel="rear_left_wheel"/>-->
+	<xacro:hinge_transmission hinge="front_right_hinge"/>
+	<xacro:hinge_transmission hinge="front_left_hinge"/>
+	<!-- Sensors -->
 	<link name="left_camera_mount">
 		<visual>
@@ -255,4 +266,5 @@
 	</link>
 	<xacro:fixed_offset_joint parent="lidar_mount" child="lidar" offset="0 0 ${lidar_mount_height}"/>
+	<!-- Link Gazebo and ROS - this has to happen as the last thing -->
 	<xacro:include filename="$(find jetsoncar_description)/urdf/gazebo.xacro" />
 </robot>

File: jetsoncar_description/urdf/joints.xacro (robot description, xacro)
@@ -8,5 +8,20 @@
 		</joint>
 	</xacro:macro>
-	<xacro:macro name="steering_joint" params="parent child offset">
+	<xacro:macro name="dampener_joint" params="parent child offset">
+		<joint name="${parent}_to_${child}" type="prismatic">
+			<parent link="${parent}"/>
+			<child link="${child}"/>
+			<origin xyz="${offset}" rpy="0 0 0" /> <!-- offset from parent to child, so with direction based in parent frame -->
+			<axis xyz="0 0 -1"/> <!-- suspension works up and down -->
+			<limit lower="${susp_lower}" upper="${susp_upper}" effort="0" velocity="0"/>
+		        <dynamics damping="${susp_damping}" spring_stiffness="${susp_stiffness}" spring_reference="${susp_spring_center}"/>
+			<physics>
+				<ode>
+					<implicit_spring_damper>0</implicit_spring_damper>
+				</ode>
+			</physics>
+		</joint>
+	</xacro:macro>
+	<xacro:macro name="hinge_joint" params="parent child offset">
 		<joint name="${child}_joint" type="revolute"> <!-- revolute is a joint with a range limited motion around its' axis -->
 			<parent link="${parent}"/>
@@ -14,8 +29,8 @@
 			<origin xyz="${offset}" rpy="0 0 0" /> <!-- offset from parent to child, so with direction based in parent frame -->
 			<axis xyz="0 0 1"/>
-	    		<limit lower="-${steering_wheel_angle_limit}" upper="${steering_wheel_angle_limit}" effort="100" velocity="0.5"/>
+	    		<limit lower="-${steering_wheel_angle_limit}" upper="${steering_wheel_angle_limit}" effort="100" velocity="0.5"/> <!-- effeort is similar to torque/acceleration -->
 			<!-- friction - The physical static friction. For prismatic joints, the units are Newtons. For revolving joints, the units are Newton meters. -->
 			<!-- damping - The physical damping value. For prismatic joints, the units are Newton seconds per meter. For revolving joints, Newton meter secons per radian. -->
-			<dynamics friction="0.0" damping="0.0"/>
+			<!--<dynamics friction="0.0" damping="0.0"/>-->
 		</joint>
 	</xacro:macro>
@@ -28,5 +43,5 @@
 			<!-- friction - The physical static friction. For prismatic joints, the units are Newtons. For revolving joints, the units are Newton meters. -->
 			<!-- damping - The physical damping value. For prismatic joints, the units are Newton seconds per meter. For revolving joints, Newton meter secons per radian. -->
-			<dynamics friction="0.0" damping="0.0"/>
+			<!--<dynamics friction="0.0" damping="0.0"/>-->
 		</joint>
 	</xacro:macro>

File: jetsoncar_description/urdf/physical.xacro (robot description, xacro)
@@ -10,4 +10,11 @@
 	<xacro:property name="wheel_thickness" value="0.064" />
 	<xacro:property name="wheel_weight" value="0.050" />
+	<!-- suspension stiffness, damping, and limits -->
+	<xacro:property name="susp_travel" value="${wheel_diameter/2}"/>
+	<xacro:property name="susp_lower" value="${-susp_travel/2}"/>
+	<xacro:property name="susp_upper" value="${susp_travel/2}"/>
+	<xacro:property name="susp_damping" value="70"/>
+	<xacro:property name="susp_stiffness" value="5"/>
+	<xacro:property name="susp_spring_center" value="0.05"/>
 	<!-- RC car physical layout -->
 	<xacro:property name="front_to_rear_wheel_center" value="0.42" />
@@ -20,4 +27,8 @@
 	<xacro:property name="baseplate_length" value="0.50" />
 	<xacro:property name="baseplate_thickness" value="0.0675" />
+	<xacro:property name="baseplate_weight" value="1.000" />
+	<!-- Shaft and mount related properties -->
+	<xacro:property name="mount_weight" value="0.500" />
+	<xacro:property name="shaft_weight" value="0.100" />
 	<!-- Camera related properties -->
 	<xacro:property name="camera_width" value="0.094" />
@@ -33,5 +44,5 @@
 	<xacro:property name="lidar_length" value="0.05" />
 	<xacro:property name="lidar_height" value="0.05" />
-	<xacro:property name="lidar_weight" value="0.250" />
+	<xacro:property name="lidar_weight" value="0.200" />
 	<xacro:property name="lidar_mount_diameter" value="0.08" />
 	<xacro:property name="lidar_mount_height" value="0.13" />
@@ -47,5 +58,5 @@
 	<xacro:macro name="imu_inertial">
 		<origin xyz="0 0 0" rpy="0 0 0" /> <!-- origin (0,0,0) is in the center of the box -->
-		<xacro:box_inertial mass="0.005" length="${imu_length}" width="${imu_width}" height="${imu_height}" />
+		<xacro:box_inertial mass="0.010" length="${imu_length}" width="${imu_width}" height="${imu_height}" /> <!-- 10 grams -->
 	</xacro:macro>
 	<!-- Baseplate -->
@@ -58,5 +69,5 @@
 	<xacro:macro name="baseplate_inertial">
 		<origin xyz="0 0 ${baseplate_thickness/2}" rpy="0 0 0" /> <!-- origin (0,0,0) is in the center of the box, so place the origin of this in the bottom of baseplate -->
-		<xacro:box_inertial mass="0.500" length="${baseplate_length}" width="${baseplate_width}" height="${baseplate_thickness}" />
+		<xacro:box_inertial mass="${baseplate_weight}" length="${baseplate_length}" width="${baseplate_width}" height="${baseplate_thickness}" />
 	</xacro:macro>
 	<!-- Mount -->
@@ -75,9 +86,9 @@
 	<xacro:macro name="front_mount_inertial">
 		<origin xyz="0 0 0" rpy="0 0.5 0" /> <!-- origin (0,0,0) is in the center of the box -->
-		<xacro:box_inertial mass="0.200" length="0.24" width="0.12" height="0.01" />
+		<xacro:box_inertial mass="${mount_weight}" length="0.24" width="0.12" height="0.01" />
 	</xacro:macro>
 	<xacro:macro name="rear_mount_inertial">
 		<origin xyz="0 0 0" rpy="0 -0.5 0" /> <!-- origin (0,0,0) is in the center of the box -->
-		<xacro:box_inertial mass="0.200" length="0.24" width="0.12" height="0.01" />
+		<xacro:box_inertial mass="${mount_weight}" length="0.24" width="0.12" height="0.01" />
 	</xacro:macro>
 	<!-- Shaft -->
@@ -90,8 +101,8 @@
 	<xacro:macro name="shaft_inertial">
 		<origin xyz="0 0 0" rpy="1.570796327 0 0" /> <!-- origin (0,0,0) is in the center of the cylinder -->
-		<xacro:cylinder_inertial mass="0.100" radius="0.018" length="${left_to_right_wheel_center}" />
+		<xacro:cylinder_inertial mass="${shaft_weight}" radius="0.018" length="${left_to_right_wheel_center}" />
 	</xacro:macro>
-	<!-- Bearing -->
-	<xacro:macro name="bearing_geometry">
+	<!-- Hinge -->
+	<xacro:macro name="hinge_geometry">
 		<origin xyz="0 0 0" rpy="0 0 0" />
 		<geometry>
@@ -99,8 +110,8 @@
 		</geometry>
 	</xacro:macro>
-	<xacro:macro name="bearing_inertial">
+	<xacro:macro name="hinge_inertial">
 		<origin xyz="0 0 0" rpy="0 0 0" />
-		<mass value="1e-5" />
-		<inertia ixx="1e-9" ixy="0" ixz="0" iyy="1e-9" iyz="0" izz="1e-9" /> <!-- small inertia -->
+		<mass value="0.01" />
+		<inertia ixx="1e-6" ixy="0" ixz="0" iyy="1e-6" iyz="0" izz="1e-6" /> <!-- small inertia -->
 	</xacro:macro>
 	<!-- Wheel -->
@@ -125,5 +136,5 @@
 		<origin xyz="0 0 0" rpy="0 0 0" /> <!-- origin (0,0,0) is in the center of the box -->
 		<mass value="0.005" /> <!-- 5 grams -->
-		<inertia ixx="1e-9" ixy="0" ixz="0" iyy="1e-9" iyz="0" izz="1e-9" /> <!-- small inertia -->
+		<inertia ixx="1e-6" ixy="0" ixz="0" iyy="1e-6" iyz="0" izz="1e-6" /> <!-- small inertia -->
 	</xacro:macro>
 	<xacro:macro name="camera_geometry">
