Commit message: Fixed inertia error + added test scripts for pushing controller commands
Inertia error caused the car to start stuck in the ground

File: jetsoncar_description/urdf/gazebo.xacro (robot description, xacro)
@@ -4,4 +4,138 @@
 	<!-- see the guide: http://wiki.ros.org/urdf/Tutorials/Using%20a%20URDF%20in%20Gazebo -->
 	<!-- inspired from https://github.com/mit-racecar/racecar-simulator/blob/master/racecar_description/urdf/racecar.gazebo and https://github.com/husky/husky_simulator/blob/indigo-devel/husky_gazebo/urdf/husky.gazebo.xacro -->
+	<!-- Visual and physical properties -->
+	<!-- See http://gazebosim.org/tutorials?tut=ros_urdf&cat=connect_ros -->
+	<gazebo reference="baseplate">
+		<mu1 value="0.0"/> <!-- Columb friction coefficient in fdir1 direction -->
+		<mu2 value="0.0"/> <!-- Columb friction in perpendicular direction to fdir1 -->
+		<kp  value="10000000.0" /> <!-- contact stiffness -->
+		<kd  value="1.0" /> <!-- contact damping -->
+		<material>Gazebo/Grey</material>
+		<!--<turnGravityOff>false</turnGravityOff>-->
+	</gazebo>
+	<gazebo reference="imu">
+		<mu1 value="0.0"/> <!-- Columb friction coefficient in fdir1 direction -->
+		<mu2 value="0.0"/> <!-- Columb friction in perpendicular direction to fdir1 -->
+		<kp  value="10000000.0" /> <!-- contact stiffness -->
+		<kd  value="1.0" /> <!-- contact damping -->
+		<material>Gazebo/Grey</material>
+		<!--<turnGravityOff>false</turnGravityOff>-->
+	</gazebo>
+	<gazebo reference="front_mount">
+		<mu1 value="0.0"/> <!-- Columb friction coefficient in fdir1 direction -->
+		<mu2 value="0.0"/> <!-- Columb friction in perpendicular direction to fdir1 -->
+		<kp  value="10000000.0" /> <!-- contact stiffness -->
+		<kd  value="1.0" /> <!-- contact damping -->
+		<material>Gazebo/Grey</material>
+		<!--<turnGravityOff>false</turnGravityOff>-->
+	</gazebo>
+	<gazebo reference="rear_mount">
+		<mu1 value="0.0"/> <!-- Columb friction coefficient in fdir1 direction -->
+		<mu2 value="0.0"/> <!-- Columb friction in perpendicular direction to fdir1 -->
+		<kp  value="10000000.0" /> <!-- contact stiffness -->
+		<kd  value="1.0" /> <!-- contact damping -->
+		<material>Gazebo/Grey</material>
+		<!--<turnGravityOff>false</turnGravityOff>-->
+	</gazebo>
+	<gazebo reference="front_shaft">
+		<mu1 value="0.0"/> <!-- Columb friction coefficient in fdir1 direction -->
+		<mu2 value="0.0"/> <!-- Columb friction in perpendicular direction to fdir1 -->
+		<kp  value="10000000.0" /> <!-- contact stiffness -->
+		<kd  value="1.0" /> <!-- contact damping -->
+		<material>Gazebo/Black</material>
+		<!--<turnGravityOff>false</turnGravityOff>-->
+	</gazebo>
+	<gazebo reference="rear_shaft">
+		<mu1 value="0.0"/> <!-- Columb friction coefficient in fdir1 direction -->
+		<mu2 value="0.0"/> <!-- Columb friction in perpendicular direction to fdir1 -->
+		<kp  value="10000000.0" /> <!-- contact stiffness -->
+		<kd  value="1.0" /> <!-- contact damping -->
+		<material>Gazebo/Black</material>
+		<!--<turnGravityOff>false</turnGravityOff>-->
+	</gazebo>
+	<gazebo reference="front_right_wheel">
+		<mu1 value="1.0"/> <!-- Columb friction coefficient in fdir1 direction -->
+		<mu2 value="1.0"/> <!-- Columb friction in perpendicular direction to fdir1 -->
+		<kp  value="10000000.0" /> <!-- contact stiffness -->
+		<kd  value="1.0" /> <!-- contact damping -->
+		<fdir1 value="1 0 0"/> <!-- direction of mu1 friction coefficient in the collision frame -->
+		<material>Gazebo/Black</material>
+		<!--<turnGravityOff>false</turnGravityOff>-->
+	</gazebo>
+	<gazebo reference="front_left_wheel">
+		<mu1 value="1.0"/> <!-- Columb friction coefficient in fdir1 direction -->
+		<mu2 value="1.0"/> <!-- Columb friction in perpendicular direction to fdir1 -->
+		<kp  value="10000000.0" /> <!-- contact stiffness -->
+		<kd  value="1.0" /> <!-- contact damping -->
+		<fdir1 value="1 0 0"/> <!-- direction of mu1 friction coefficient in the collision frame -->
+		<material>Gazebo/Black</material>
+		<!--<turnGravityOff>false</turnGravityOff>-->
+	</gazebo>
+	<gazebo reference="rear_right_wheel">
+		<mu1 value="1.0"/> <!-- Columb friction coefficient in fdir1 direction -->
+		<mu2 value="1.0"/> <!-- Columb friction in perpendicular direction to fdir1 -->
+		<kp  value="10000000.0" /> <!-- contact stiffness -->
+		<kd  value="1.0" /> <!-- contact damping -->
+		<fdir1 value="1 0 0"/> <!-- direction of mu1 friction coefficient in the collision frame -->
+		<material>Gazebo/Black</material>
+		<!--<turnGravityOff>false</turnGravityOff>-->
+	</gazebo>
+	<gazebo reference="rear_left_wheel">
+		<mu1 value="1.0"/> <!-- Columb friction coefficient in fdir1 direction -->
+		<mu2 value="1.0"/> <!-- Columb friction in perpendicular direction to fdir1 -->
+		<kp  value="10000000.0" /> <!-- contact stiffness -->
+		<kd  value="1.0" /> <!-- contact damping -->
+		<fdir1 value="1 0 0"/> <!-- direction of mu1 friction coefficient in the collision frame -->
+		<material>Gazebo/Black</material>
+		<!--<turnGravityOff>false</turnGravityOff>-->
+	</gazebo>
+	<gazebo reference="lidar_mount">
+		<mu1 value="0.0"/> <!-- Columb friction coefficient in fdir1 direction -->
+		<mu2 value="0.0"/> <!-- Columb friction in perpendicular direction to fdir1 -->
+		<kp  value="10000000.0" /> <!-- contact stiffness -->
+		<kd  value="1.0" /> <!-- contact damping -->
+		<material>Gazebo/Red</material>
+		<!--<turnGravityOff>false</turnGravityOff>-->
+	</gazebo>
+	<gazebo reference="lidar">
+		<mu1 value="0.0"/> <!-- Columb friction coefficient in fdir1 direction -->
+		<mu2 value="0.0"/> <!-- Columb friction in perpendicular direction to fdir1 -->
+		<kp  value="10000000.0" /> <!-- contact stiffness -->
+		<kd  value="1.0" /> <!-- contact damping -->
+		<material>Gazebo/Black</material>
+		<!--<turnGravityOff>false</turnGravityOff>-->
+	</gazebo>
+	<gazebo reference="left_camera_mount">
+		<mu1 value="0.0"/> <!-- Columb friction coefficient in fdir1 direction -->
+		<mu2 value="0.0"/> <!-- Columb friction in perpendicular direction to fdir1 -->
+		<kp  value="10000000.0" /> <!-- contact stiffness -->
+		<kd  value="1.0" /> <!-- contact damping -->
+		<material>Gazebo/Black</material>
+		<!--<turnGravityOff>false</turnGravityOff>-->
+	</gazebo>
+	<gazebo reference="left_camera">
+		<mu1 value="0.0"/> <!-- Columb friction coefficient in fdir1 direction -->
+		<mu2 value="0.0"/> <!-- Columb friction in perpendicular direction to fdir1 -->
+		<kp  value="10000000.0" /> <!-- contact stiffness -->
+		<kd  value="1.0" /> <!-- contact damping -->
+		<material>Gazebo/Blue</material>
+		<!--<turnGravityOff>false</turnGravityOff>-->
+	</gazebo>
+	<gazebo reference="right_camera_mount">
+		<mu1 value="0.0"/> <!-- Columb friction coefficient in fdir1 direction -->
+		<mu2 value="0.0"/> <!-- Columb friction in perpendicular direction to fdir1 -->
+		<kp  value="10000000.0" /> <!-- contact stiffness -->
+		<kd  value="1.0" /> <!-- contact damping -->
+		<material>Gazebo/Black</material>
+		<!--<turnGravityOff>false</turnGravityOff>-->
+	</gazebo>
+	<gazebo reference="right_camera">
+		<mu1 value="0.0"/> <!-- Columb friction coefficient in fdir1 direction -->
+		<mu2 value="0.0"/> <!-- Columb friction in perpendicular direction to fdir1 -->
+		<kp  value="10000000.0" /> <!-- contact stiffness -->
+		<kd  value="1.0" /> <!-- contact damping -->
+		<material>Gazebo/Blue</material>
+		<!--<turnGravityOff>false</turnGravityOff>-->
+	</gazebo>
 	<!-- We need to link Gazebo and ROS and let Gazebo load all the previously defined ROS parameters. Therefore this Gazebo file should be included in the end of the main xacro file! -->
 	<!-- Link Gazebo and ROS -->
@@ -9,152 +143,6 @@
 		<plugin name="gazebo_ros_control" filename="libgazebo_ros_control.so">
 			<robotNamespace>/jetsoncar</robotNamespace>
-			<!--<robotSimType>gazebo_ros_control/DefaultRobotHWSim</robotSimType> -->
+			<robotSimType>gazebo_ros_control/DefaultRobotHWSim</robotSimType>
 		</plugin>
-	</gazebo>
-	<!-- Visual and physical properties -->
-	<!-- See http://gazebosim.org/tutorials?tut=ros_urdf&cat=connect_ros -->
-	<gazebo reference="baseplate">
-		<material>Gazebo/Grey</material>
-		<mu1 value="0.0"/> <!-- Columb friction coefficient in fdir1 direction -->
-		<mu2 value="0.0"/> <!-- Columb friction in perpendicular direction to fdir1 -->
-		<fdir1 value="1 0 0"/> <!-- direction of mu1 friction coefficient in the collision frame -->
-		<kp  value="10000000.0" /> <!-- contact stiffness -->
-		<kd  value="1.0" /> <!-- contact damping -->
-		<turnGravityOff>false</turnGravityOff>
-	</gazebo>
-	<gazebo reference="imu">
-		<material>Gazebo/Grey</material>
-		<mu1 value="0.0"/> <!-- Columb friction coefficient in fdir1 direction -->
-		<mu2 value="0.0"/> <!-- Columb friction in perpendicular direction to fdir1 -->
-		<fdir1 value="1 0 0"/> <!-- direction of mu1 friction coefficient in the collision frame -->
-		<kp  value="10000000.0" /> <!-- contact stiffness -->
-		<kd  value="1.0" /> <!-- contact damping -->
-		<turnGravityOff>false</turnGravityOff>
-	</gazebo>
-	<gazebo reference="front_mount">
-		<material>Gazebo/Grey</material>
-		<mu1 value="0.0"/> <!-- Columb friction coefficient in fdir1 direction -->
-		<mu2 value="0.0"/> <!-- Columb friction in perpendicular direction to fdir1 -->
-		<fdir1 value="1 0 0"/> <!-- direction of mu1 friction coefficient in the collision frame -->
-		<kp  value="10000000.0" /> <!-- contact stiffness -->
-		<kd  value="1.0" /> <!-- contact damping -->
-		<turnGravityOff>false</turnGravityOff>
-	</gazebo>
-	<gazebo reference="rear_mount">
-		<material>Gazebo/Grey</material>
-		<mu1 value="0.0"/> <!-- Columb friction coefficient in fdir1 direction -->
-		<mu2 value="0.0"/> <!-- Columb friction in perpendicular direction to fdir1 -->
-		<fdir1 value="1 0 0"/> <!-- direction of mu1 friction coefficient in the collision frame -->
-		<kp  value="10000000.0" /> <!-- contact stiffness -->
-		<kd  value="1.0" /> <!-- contact damping -->
-		<turnGravityOff>false</turnGravityOff>
-	</gazebo>
-	<gazebo reference="front_shaft">
-		<material>Gazebo/Black</material>
-		<mu1 value="0.0"/> <!-- Columb friction coefficient in fdir1 direction -->
-		<mu2 value="0.0"/> <!-- Columb friction in perpendicular direction to fdir1 -->
-		<fdir1 value="1 0 0"/> <!-- direction of mu1 friction coefficient in the collision frame -->
-		<kp  value="10000000.0" /> <!-- contact stiffness -->
-		<kd  value="1.0" /> <!-- contact damping -->
-		<turnGravityOff>false</turnGravityOff>
-	</gazebo>
-	<gazebo reference="rear_shaft">
-		<material>Gazebo/Black</material>
-		<mu1 value="0.0"/> <!-- Columb friction coefficient in fdir1 direction -->
-		<mu2 value="0.0"/> <!-- Columb friction in perpendicular direction to fdir1 -->
-		<fdir1 value="1 0 0"/> <!-- direction of mu1 friction coefficient in the collision frame -->
-		<kp  value="10000000.0" /> <!-- contact stiffness -->
-		<kd  value="1.0" /> <!-- contact damping -->
-		<turnGravityOff>false</turnGravityOff>
-	</gazebo>
-	<gazebo reference="front_right_wheel">
-		<material>Gazebo/Black</material>
-		<mu1 value="1.0"/> <!-- Columb friction coefficient in fdir1 direction -->
-		<mu2 value="1.0"/> <!-- Columb friction in perpendicular direction to fdir1 -->
-		<fdir1 value="1 0 0"/> <!-- direction of mu1 friction coefficient in the collision frame -->
-		<kp  value="10000000.0" /> <!-- contact stiffness -->
-		<kd  value="1.0" /> <!-- contact damping -->
-		<turnGravityOff>false</turnGravityOff>
-	</gazebo>
-	<gazebo reference="front_left_wheel">
-		<material>Gazebo/Black</material>
-		<mu1 value="1.0"/> <!-- Columb friction coefficient in fdir1 direction -->
-		<mu2 value="1.0"/> <!-- Columb friction in perpendicular direction to fdir1 -->
-		<fdir1 value="1 0 0"/> <!-- direction of mu1 friction coefficient in the collision frame -->
-		<kp  value="10000000.0" /> <!-- contact stiffness -->
-		<kd  value="1.0" /> <!-- contact damping -->
-		<turnGravityOff>false</turnGravityOff>
-	</gazebo>
-	<gazebo reference="rear_right_wheel">
-		<material>Gazebo/Black</material>
-		<mu1 value="1.0"/> <!-- Columb friction coefficient in fdir1 direction -->
-		<mu2 value="1.0"/> <!-- Columb friction in perpendicular direction to fdir1 -->
-		<fdir1 value="1 0 0"/> <!-- direction of mu1 friction coefficient in the collision frame -->
-		<kp  value="10000000.0" /> <!-- contact stiffness -->
-		<kd  value="1.0" /> <!-- contact damping -->
-		<turnGravityOff>false</turnGravityOff>
-	</gazebo>
-	<gazebo reference="rear_left_wheel">
-		<material>Gazebo/Black</material>
-		<mu1 value="1.0"/> <!-- Columb friction coefficient in fdir1 direction -->
-		<mu2 value="1.0"/> <!-- Columb friction in perpendicular direction to fdir1 -->
-		<fdir1 value="1 0 0"/> <!-- direction of mu1 friction coefficient in the collision frame -->
-		<kp  value="10000000.0" /> <!-- contact stiffness -->
-		<kd  value="1.0" /> <!-- contact damping -->
-		<turnGravityOff>false</turnGravityOff>
-	</gazebo>
-	<gazebo reference="lidar_mount">
-		<material>Gazebo/Red</material>
-		<mu1 value="0.0"/> <!-- Columb friction coefficient in fdir1 direction -->
-		<mu2 value="0.0"/> <!-- Columb friction in perpendicular direction to fdir1 -->
-		<fdir1 value="1 0 0"/> <!-- direction of mu1 friction coefficient in the collision frame -->
-		<kp  value="10000000.0" /> <!-- contact stiffness -->
-		<kd  value="1.0" /> <!-- contact damping -->
-		<turnGravityOff>false</turnGravityOff>
-	</gazebo>
-	<gazebo reference="lidar">
-		<material>Gazebo/Black</material>
-		<mu1 value="0.0"/> <!-- Columb friction coefficient in fdir1 direction -->
-		<mu2 value="0.0"/> <!-- Columb friction in perpendicular direction to fdir1 -->
-		<fdir1 value="1 0 0"/> <!-- direction of mu1 friction coefficient in the collision frame -->
-		<kp  value="10000000.0" /> <!-- contact stiffness -->
-		<kd  value="1.0" /> <!-- contact damping -->
-		<turnGravityOff>false</turnGravityOff>
-	</gazebo>
-	<gazebo reference="left_camera_mount">
-		<material>Gazebo/Black</material>
-		<mu1 value="0.0"/> <!-- Columb friction coefficient in fdir1 direction -->
-		<mu2 value="0.0"/> <!-- Columb friction in perpendicular direction to fdir1 -->
-		<fdir1 value="1 0 0"/> <!-- direction of mu1 friction coefficient in the collision frame -->
-		<kp  value="10000000.0" /> <!-- contact stiffness -->
-		<kd  value="1.0" /> <!-- contact damping -->
-		<turnGravityOff>false</turnGravityOff>
-	</gazebo>
-	<gazebo reference="left_camera">
-		<material>Gazebo/Blue</material>
-		<mu1 value="0.0"/> <!-- Columb friction coefficient in fdir1 direction -->
-		<mu2 value="0.0"/> <!-- Columb friction in perpendicular direction to fdir1 -->
-		<fdir1 value="1 0 0"/> <!-- direction of mu1 friction coefficient in the collision frame -->
-		<kp  value="10000000.0" /> <!-- contact stiffness -->
-		<kd  value="1.0" /> <!-- contact damping -->
-		<turnGravityOff>false</turnGravityOff>
-	</gazebo>
-	<gazebo reference="right_camera_mount">
-		<material>Gazebo/Black</material>
-		<mu1 value="0.0"/> <!-- Columb friction coefficient in fdir1 direction -->
-		<mu2 value="0.0"/> <!-- Columb friction in perpendicular direction to fdir1 -->
-		<fdir1 value="1 0 0"/> <!-- direction of mu1 friction coefficient in the collision frame -->
-		<kp  value="10000000.0" /> <!-- contact stiffness -->
-		<kd  value="1.0" /> <!-- contact damping -->
-		<turnGravityOff>false</turnGravityOff>
-	</gazebo>
-	<gazebo reference="right_camera">
-		<material>Gazebo/Blue</material>
-		<mu1 value="0.0"/> <!-- Columb friction coefficient in fdir1 direction -->
-		<mu2 value="0.0"/> <!-- Columb friction in perpendicular direction to fdir1 -->
-		<fdir1 value="1 0 0"/> <!-- direction of mu1 friction coefficient in the collision frame -->
-		<kp  value="10000000.0" /> <!-- contact stiffness -->
-		<kd  value="1.0" /> <!-- contact damping -->
-		<turnGravityOff>false</turnGravityOff>
 	</gazebo>
 	<!-- Plugins, eg. sensors -->

File: jetsoncar_description/urdf/jetsoncar.xacro (robot description, xacro)
@@ -13,5 +13,4 @@
 	<!-- X axis direction is forward, Y axis direction is left -->
 	<xacro:include filename="$(find jetsoncar_description)/urdf/functions.xacro" />
-	<xacro:include filename="$(find jetsoncar_description)/urdf/materials.xacro" />
 	<xacro:include filename="$(find jetsoncar_description)/urdf/physical.xacro" />
 	<xacro:include filename="$(find jetsoncar_description)/urdf/joints.xacro" />
@@ -103,7 +102,7 @@
 			<xacro:hinge_geometry/>
 		</visual>
-		<collision>
-			<xacro:hinge_geometry/>
-		</collision>
+		<!--<collision>
+			<xacro:hinge_geometry/>
+		</collision>-->
 		<inertial>
 			<xacro:hinge_inertial/>
@@ -111,4 +110,5 @@
 	</link>
 	<xacro:hinge_joint parent="front_shaft" child="front_right_hinge" offset="0 -${left_to_right_wheel_center/2} 0"/>
+	<xacro:hinge_transmission hinge="front_right_hinge"/>
 	<link name="front_left_hinge">
 		<visual>
@@ -116,7 +116,7 @@
 			<xacro:hinge_geometry/>
 		</visual>
-		<collision>
-			<xacro:hinge_geometry/>
-		</collision>
+		<!--<collision>
+			<xacro:hinge_geometry/>
+		</collision>-->
 		<inertial>
 			<xacro:hinge_inertial/>
@@ -124,4 +124,5 @@
 	</link>
 	<xacro:hinge_joint parent="front_shaft" child="front_left_hinge" offset="0 ${left_to_right_wheel_center/2} 0"/>
+	<xacro:hinge_transmission hinge="front_left_hinge"/>
 	<link name="front_right_wheel">
 		<visual>
@@ -131,5 +132,5 @@
 		<collision>
 			<xacro:wheel_geometry/>
-			<contact_coefficients mu="0" kp="1000.0" kd="1.0"/>  <!-- mu=The friction coefficient, kp=Stiffness coefficient, kd=Dampening coefficient -->
+			<!--<contact_coefficients mu="0" kp="1000.0" kd="1.0"/>-->  <!-- mu=The friction coefficient, kp=Stiffness coefficient, kd=Dampening coefficient -->
 		</collision>
 		<inertial>
@@ -138,4 +139,5 @@
 	</link>
 	<xacro:wheel_joint parent="front_right_hinge" child="front_right_wheel" offset="0 0 0"/>
+	<xacro:wheel_transmission wheel="front_right_wheel"/>
 	<link name="front_left_wheel">
 		<visual>
@@ -145,5 +147,5 @@
 		<collision>
 			<xacro:wheel_geometry/>
-			<contact_coefficients mu="0" kp="1000.0" kd="1.0"/>  <!-- mu=The friction coefficient, kp=Stiffness coefficient, kd=Dampening coefficient -->
+			<!--<contact_coefficients mu="0" kp="1000.0" kd="1.0"/>-->  <!-- mu=The friction coefficient, kp=Stiffness coefficient, kd=Dampening coefficient -->
 		</collision>
 		<inertial>
@@ -152,4 +154,5 @@
 	</link>
 	<xacro:wheel_joint parent="front_left_hinge" child="front_left_wheel" offset="0 0 0"/>
+	<xacro:wheel_transmission wheel="front_left_wheel"/>
 	<link name="rear_right_wheel">
 		<visual>
@@ -159,5 +162,5 @@
 		<collision>
 			<xacro:wheel_geometry/>
-			<contact_coefficients mu="0" kp="1000.0" kd="1.0"/>  <!-- mu=The friction coefficient, kp=Stiffness coefficient, kd=Dampening coefficient -->
+			<!--<contact_coefficients mu="0" kp="1000.0" kd="1.0"/>-->  <!-- mu=The friction coefficient, kp=Stiffness coefficient, kd=Dampening coefficient -->
 		</collision>
 		<inertial>
@@ -166,4 +169,5 @@
 	</link>
 	<xacro:wheel_joint parent="rear_shaft" child="rear_right_wheel" offset="0 -${left_to_right_wheel_center/2} 0"/>
+	<!--<xacro:wheel_transmission wheel="rear_right_wheel"/>-->
 	<link name="rear_left_wheel">
 		<visual>
@@ -173,5 +177,5 @@
 		<collision>
 			<xacro:wheel_geometry/>
-			<contact_coefficients mu="0" kp="1000.0" kd="1.0"/>  <!-- mu=The friction coefficient, kp=Stiffness coefficient, kd=Dampening coefficient -->
+			<!--<contact_coefficients mu="0" kp="1000.0" kd="1.0"/>-->  <!-- mu=The friction coefficient, kp=Stiffness coefficient, kd=Dampening coefficient -->
 		</collision>
 		<inertial>
@@ -180,11 +184,5 @@
 	</link>
 	<xacro:wheel_joint parent="rear_shaft" child="rear_left_wheel" offset="0 ${left_to_right_wheel_center/2} 0"/>
-	<!-- Transmissions are motors attached to a certain joint. We thus need to instantiate transmissions at the corresponding joints -->
-	<xacro:wheel_transmission wheel="front_right_wheel"/>
-	<xacro:wheel_transmission wheel="front_left_wheel"/>
-	<!--<xacro:wheel_transmission wheel="rear_right_wheel"/>    Currently only front wheel drive!
-	<xacro:wheel_transmission wheel="rear_left_wheel"/>-->
-	<xacro:hinge_transmission hinge="front_right_hinge"/>
-	<xacro:hinge_transmission hinge="front_left_hinge"/>
+	<!--<xacro:wheel_transmission wheel="rear_left_wheel"/>-->
 	<!-- Sensors -->
 	<link name="left_camera_mount">
@@ -268,3 +266,4 @@
 	<!-- Link Gazebo and ROS - this has to happen as the last thing -->
 	<xacro:include filename="$(find jetsoncar_description)/urdf/gazebo.xacro" />
+	<xacro:include filename="$(find jetsoncar_description)/urdf/materials.xacro" />
 </robot>

File: jetsoncar_description/urdf/joints.xacro (robot description, xacro)
@@ -29,5 +29,5 @@
 			<origin xyz="${offset}" rpy="0 0 0" /> <!-- offset from parent to child, so with direction based in parent frame -->
 			<axis xyz="0 0 1"/>
-	    		<limit lower="-${steering_wheel_angle_limit}" upper="${steering_wheel_angle_limit}" effort="100" velocity="0.5"/> <!-- effeort is similar to torque/acceleration -->
+	    		<limit lower="-${steering_wheel_angle_limit}" upper="${steering_wheel_angle_limit}" effort="10" velocity="100"/> <!-- effeort is similar to torque/acceleration -->
 			<!-- friction - The physical static friction. For prismatic joints, the units are Newtons. For revolving joints, the units are Newton meters. -->
 			<!-- damping - The physical damping value. For prismatic joints, the units are Newton seconds per meter. For revolving joints, Newton meter secons per radian. -->
@@ -44,4 +44,5 @@
 			<!-- damping - The physical damping value. For prismatic joints, the units are Newton seconds per meter. For revolving joints, Newton meter secons per radian. -->
 			<!--<dynamics friction="0.0" damping="0.0"/>-->
+			<limit effort="10" velocity="100"/>
 		</joint>
 	</xacro:macro>

File: jetsoncar_description/urdf/physical.xacro (robot description, xacro)
@@ -9,5 +9,5 @@
 	<xacro:property name="wheel_diameter" value="0.155" />
 	<xacro:property name="wheel_thickness" value="0.064" />
-	<xacro:property name="wheel_weight" value="0.050" />
+	<xacro:property name="wheel_weight" value="0.150" />
 	<!-- suspension stiffness, damping, and limits -->
 	<xacro:property name="susp_travel" value="${wheel_diameter/2}"/>
@@ -112,5 +112,5 @@
 	<xacro:macro name="hinge_inertial">
 		<origin xyz="0 0 0" rpy="0 0 0" />
-		<mass value="0.01" />
+		<mass value="0.05" />
 		<inertia ixx="1e-6" ixy="0" ixz="0" iyy="1e-6" iyz="0" izz="1e-6" /> <!-- small inertia -->
 	</xacro:macro>
